Commit message: try to make sonar spin by unsuccesful

File: rover_description/urdf/rover.xacro (robot description, xacro)
@@ -149,10 +149,20 @@
     <joint_properties damping="1.0" friction="1.0"/>
   </joint>
-  <joint name="sonar_front_joint" type="fixed">
-      <axis xyz="0 1 0" />
-      <origin rpy="0 0 0" xyz="0.5 0 0.25" />
+  <joint name="sonar_front_joint" type="continuous">
+      <axis xyz="0 0 1" />
+      <origin rpy="0 0 0" xyz="0 0 0.35" />
       <parent link="base_footprint"/>
       <child link="base_sonar_front"/>
   </joint>
+  <transmission name="sonar_trans" type="SimpleTransmission">
+    <type>transmission_interface/SimpleTransmission</type>
+    <actuator name="sonar_motor">
+      <hardwareInterface>hardware_interface/EffortJointInterface</hardwareInterface>
+    <mechanicalReduction>1</mechanicalReduction>
+    </actuator>
+    <joint name="sonar_front_joint">
+      <hardwareInterface>hardware_interface/EffortJointInterface</hardwareInterface>
+    </joint>
+  </transmission>
   <link name="base_sonar_front">
       <collision>
@@ -174,4 +184,11 @@
       </inertial>
   </link>
+  <gazebo>
+    <plugin name="gazebo_ros_control" filename="libgazebo_ros_control.so">
+      <robotNamespace>/Rover</robotNamespace>
+      <controlPeriod>0.1</controlPeriod>
+      <!-- <legacyModeNS>false</legacyModeNS> -->
+    </plugin>
+  </gazebo>
   <link name="dummy">
   </link>

Commit message: modify inertia, pid parameter and control period

File: rover_description/urdf/rover.xacro (robot description, xacro)
@@ -9,10 +9,10 @@
       <origin xyz="0.0 0 0.1" rpy=" 0 0 0"/>
       <inertia
-          ixx="0.1"
+          ixx="1000"
           ixy="0"
           ixz="0"
-          iyy="0.1"
+          iyy="1000"
           iyz="0"
-          izz="0.1"/>
+          izz="100"/>
     </inertial>
     <collision name='collision'>
@@ -181,5 +181,5 @@
         <mass value="1e-5" />
         <origin xyz="0 0 0" rpy="0 0 0"/>
-        <inertia ixx="1e-6" ixy="0" ixz="0" iyy="1e-6" iyz="0" izz="1e-6" />
+        <inertia ixx="10" ixy="0" ixz="0" iyy="10" iyz="0" izz="1" />
       </inertial>
   </link>
@@ -187,5 +187,5 @@
     <plugin name="gazebo_ros_control" filename="libgazebo_ros_control.so">
       <robotNamespace>/Rover</robotNamespace>
-      <controlPeriod>0.1</controlPeriod>
+      <controlPeriod>0.01</controlPeriod>
       <!-- <legacyModeNS>false</legacyModeNS> -->
     </plugin>
